File: tft_jig/tft_jig.sch (EAGLE design)
At the start: 23 parts, among them J1 SPI, J2 PJ-030DH-SMT-TR, U1 CD74HC238PWR, U2 74HC4051, U3 LM2576SX-5.0/NOPB

Commit message: fix vcc cap
Parts:
- C4: value 1mF -> 0.1uF
Changed lines of the file:
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@@
 <part name="SUPPLY21" library="scono" deviceset="GND" device=""/>
 <part name="SUPPLY22" library="scono" deviceset="GND" device=""/>
-<part name="C4" library="scono" deviceset="CAP" device="0603-CAP" value="1mF"/>
+<part name="C4" library="scono" deviceset="CAP" device="0603-CAP" value="0.1uF"/>
 <part name="SUPPLY23" library="scono" deviceset="GND" device=""/>
 <part name="C3" library="scono" deviceset="UWT0J102MNL1GS" device="" value="1mF"/>
